File: 04_USB7206Core.kicad_sch (KiCad schematic)
At the start: 0 parts

Commit message: Updated sheets to A3, added core IC, power rails, decoupling caps and USB Bus defs
Parts:
- added C1, C38: 4.7uF, symbol Device:C
- added C10, C12, C14, C16, C18, C22, C24, C26, C28, C3, C30, C32, C34, C36, C4, C6, C8: 1nF, symbol Device:C
- added C11, C13, C15, C17, C19, C2, C23, C25, C27, C29, C31, C33, C35, C37, C5, C7, C9: 100nF, symbol Device:C
- added R1, R2, R3: 10K, symbol Device:R
- added R4: 12K, symbol Device:R
- added U1: (no value), Package_DFN_QFN:VQFN-100-1EP_12x12mm_P0.4mm_EP8x8mm, symbol EW.HW.KiCADLibsSymbol:USB7206/KDX
Connections:
- new net: R4.1, U1.100 (RBIAS)
- new net +1V1: C1.1, C10.1, C11.1, C12.1, C13.1, C14.1, C15.1, C16.1, C17.1, C18.1, C19.1, C2.1, C3.1, C4.1, C5.1, C6.1, C7.1, C8.1, C9.1, U1.18 (VCORE), U1.25 (VCORE), U1.31 (VCORE), U1.38 (VCORE), U1.55 (VCORE), U1.78 (VCORE), U1.85 (VCORE), U1.9 (VCORE), U1.93 (VCORE)
- new net +3V3: C22.1, C23.1, C24.1, C25.1, C26.1, C27.1, C28.1, C29.1, C30.1, C31.1, C32.1, C33.1, C34.1, C35.1, C36.1, C37.1, C38.1, R1.1, R2.1, R3.1, U1.26 (VDD33), U1.43 (VDD33), U1.53 (VDD33), U1.62 (VDD33), U1.67 (VDD33), U1.79 (VDD33), U1.88 (VDD33), U1.99 (VDD33)
- new net GND: C1.2, C10.2, C11.2, C12.2, C13.2, C14.2, C15.2, C16.2, C17.2, C18.2, C19.2, C2.2, C22.2, C23.2, C24.2, C25.2, C26.2, C27.2, C28.2, C29.2, C3.2, C30.2, C31.2, C32.2, C33.2, C34.2, C35.2, C36.2, C37.2, C38.2, C4.2, C5.2, C6.2, C7.2, C8.2, C9.2, R4.2, U1.101 (VSS), U1.24 (TESTEN)
- new net TEST1: R1.2, U1.63 (TEST1)
- new net TEST2: R2.2, U1.64 (TEST2)
- new net TEST3: R3.2, U1.65 (TEST3)
- new net USB2DN_DM: U1.15 (USB2DN_DM2), U1.28 (USB2DN_DM3), U1.35 (USB2DN_DM4), U1.41 (USB2DN_DM6), U1.6 (USB2DN_DM1), U1.82 (USB2DN_DM5)
- new net USB2DN_DP: U1.14 (USB2DN_DP2), U1.27 (USB2DN_DP3), U1.34 (USB2DN_DP4), U1.42 (USB2DN_DP6), U1.5 (USB2DN_DP1), U1.81 (USB2DN_DP5)
- new net USB2UP_DM: U1.90 (UDB2UP_DM)
- new net USB2UP_DP: U1.89 (USB2UP_DP)
- new net USB3DN_RXDM: U1.11 (USB3DN_RXDM1), U1.20 (USB3DN_RXDM2), U1.33 (USB3DN_RXDM3), U1.40 (USB3DN_RXDM4), U1.87 (USB3DN_RXDM5)
- new net USB3DN_RXDP: U1.10 (USB3DN_RXDP1), U1.19 (USB3DN_RXDP2), U1.32 (USB3DN_RXDP3), U1.39 (USB3DN_RXDP4), U1.86 (USB3DN_RXDP5)
- new net USB3DN_TXDM: U1.17 (USB3DN_TXDM2), U1.30 (USB3DN_TXDM3), U1.37 (USB3DN_TXDM4), U1.8 (USB3DN_TXDM1), U1.84 (USB3DN_TXDM5)
- new net USB3DN_TXDP: U1.16 (USB3DN_TXDP2), U1.29 (USB3DN_TXDP3), U1.36 (USB3DN_TXDP4), U1.7 (USB3DN_TXDP1), U1.83 (USB3DN_TXDP5)
- new net USB3UP_RXDM: U1.95 (USB3UP_RXDM)
- new net USB3UP_RXDP: U1.94 (USB3UP_RXDP)
- new net USB3UP_TXDM: U1.92 (USB3UP_TXDM)
- new net USB3UP_TXDP: U1.91 (USB3UP_TXDP)
- no-connect marks 0 -> 5
Other:
- note added: "Place close to IC with low Z conn to GND"
