File: EW.HW.DeskHub1A.kicad_sch (KiCad schematic)
At the start: 0 parts

Commit message: Hardware spec and sheet structure
Other:
- added sheet 00_TopLevel (00_TopLevel.kicad_sch)
Changed lines of the file:
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@@
 	(generator_version "10.0")
 	(paper "A4")
+	(sheet
+		(at 88.9 50.8)
+		(size 114.3 63.5)
+		(exclude_from_sim no)
+		(in_bom yes)
+		(on_board yes)
+		(dnp no)
+		(fields_autoplaced yes)
+		(stroke
+			(width 0.1524)
+			(type solid)
+		)
+		(fill
+			(color 0 0 0 0)
+		)
+		(property "Sheetname" "00_TopLevel"
+			(at 88.9 50.0884 0)
+			(show_name no)
+			(do_not_autoplace no)
+			(effects
+				(font
+					(size 1.27 1.27)
+				)
+				(justify left bottom)
+			)
+		)
+		(property "Sheetfile" "00_TopLevel.kicad_sch"
+			(at 88.9 114.8846 0)
+			(show_name no)
+			(do_not_autoplace no)
+			(effects
+				(font
+					(size 1.27 1.27)
+				)
+				(justify left top)
+			)
+		)
+		(instances
+			(project "EW.HW.DeskHub1A"
+				(path "/65fce0e0-5101-4e3f-b581-6a8378cbf342"
+					(page "2")
+				)
+			)
+		)
+	)
 	(sheet_instances
 		(path "/"
